Commit message: faking an extra rotation joint.

File: config/stretch.urdf.xacro (robot description, xacro)
@@ -4,4 +4,20 @@
     <!-- Import stretch urdf file -->
     <xacro:include filename="$(find stretch_description)/urdf/stretch.urdf" />
+    <!-- This added sections seems to confuse things so ignore it -->
+    <!-- We add another fake link between odom and base-link -->
+    <link name="fake_turn_link"/>
+    <joint name="base_turn" type="revolute">
+        <limit effort="100.0" lower="-3.14" upper="3.14" velocity="1.0"/>
+        <parent link="fake_turn_link"/>
+        <child link="base_link"/>
+        <axis xyz="0 0 1"/>
+    </joint>
+    <!-- <link name="odom">
+    </link>
+    <joint name="position" type="planar">
+        <parent link="odom"/>
+        <child link="base_link"/>
+        <axis xyz="0 0 1"/>
+    </joint> -->
     <!-- Import control_xacro -->
     <xacro:include filename="stretch.ros2_control.xacro" />
